Commit message: Fixed Prismatic Joint Added Group Joint Control
Previously the sliding joint that connects the leg to the test stand was locked to be stationary. This joint is supposed to slide up and down freely to be able to test different leg behavior. Through changing the axis of movement, and increasing the allowed bounds of movement, desired behavior was achieved.

Added a Group Joint Trajectory Controller - all joints can now be controlled from a single ROS message, which makes it a little clearer/easier to control. Furthermore, this interface better suits following a desired trajectory, which is more in line with how we want to plan gait.

File: simulation/teststandv2_description/urdf/teststandv2.xacro (robot description, xacro)
@@ -114,6 +114,6 @@
   <parent link="base_link"/>
   <child link="slider_1"/>
-  <axis xyz="0.0 -1.0 0.0"/>
-  <limit effort="100" lower="0.0" upper="0.0" velocity="100"/>
+  <axis xyz="0.0 0 1"/>
+  <limit effort="100" lower="-1" upper="1" velocity="100"/>
 </joint>
 <joint name="l1" type="continuous">
